File: KiCad/PCB Rover Autonome.kicad_sch (KiCad schematic)
At the start: 0 parts

Commit message: Init library
Parts:
- added U1: STM32F410RBTx, Package_QFP:LQFP-64_10x10mm_P0.5mm, symbol PayloadLibrary:STM32F410RBTx
Connections:
- new net: U1.18 (VSS), U1.31 (VSS), U1.47 (VSS), U1.63 (VSS)
Other:
- added sheet IO Misc (io_misc.kicad_sch)
- added sheet Power (power.kicad_sch)
- added sheet Sensors (sensors.kicad_sch)
