File: KiCad/PCB Rover Autonome.kicad_sch (KiCad schematic)
At the start: 0 parts

Commit message: update fichiers pcb
Parts:
- added Accel1: BNO055, BNO055:LGA28R50P4X10_380X520X100, symbol BNO055:BNO055
- added Alti1, Alti2: MS583702BA01-50, MS583702BA01_50:XDCR_MS583702BA01-50, symbol MS583702BA01-50:MS583702BA01-50
- added Temp1: MS580301BA01-00, MS5803-01BA01_TEC, symbol 2026-01-09_20-09-59:MS580301BA01-00
- added U1: ADXL382-2BCCZ-RL7, ADXL382_2BCCZ_RL7:XDCR_ADXL382-2BCCZ-RL7, symbol ADXL382-2BCCZ-RL7:ADXL382-2BCCZ-RL7
- added U2: L76L-M33, L76L_M33:XCVR_L76L-M33, symbol L76L-M33:L76L-M33
